File: dante-audio-board.kicad_sch (KiCad schematic)
At the start: 0 parts

Commit message: start block diagram
Other:
- added sheet clock-generation (clock-generation.kicad_sch)
- added sheet sbc-header (sbc-header.kicad_sch)
Changed lines of the file:
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@@
-(kicad_sch (version 20230121) (generator eeschema)
-  (paper "A4")
-  (sheet_instances
-    (path "/" (page "1"))
-  )
+(kicad_sch
+	(version 20231120)
+	(generator "eeschema")
+	(generator_version "8.0")
+	(paper "A4")
+	(sheet
+		(at 46.99 46.99)
+		(size 12.7 64.77)
+		(fields_autoplaced yes)
+		(stroke
+			(width 0.1524)
+			(type solid)
+		)
+		(fill
+			(color 0 0 0 0.0000)
+		)
+		(property "Sheetname" "sbc-header"
+			(at 46.99 46.2784 0)
+			(effects
+				(font
+					(size 1.27 1.27)
+				)
+				(justify left bottom)
+			)
+		)
+		(property "Sheetfile" "sbc-header.kicad_sch"
+			(at 46.99 112.3446 0)
+			(effects
+				(font
+					(size 1.27 1.27)
+				)
+				(justify left top)
+			)
+		)
+		(instances
+			(project "dante-audio-board"
+				(path "/df100556-b288-4cb1-b69f-c0734132cb90"
+					(page "2")
+				)
+			)
+		)
+	)
+	(sheet
+		(at 78.74 46.99)
+		(size 40.64 24.13)
+		(fields_autoplaced yes)
+		(stroke
+			(width 0.1524)
+			(type solid)
+		)
+		(fill
+			(color 0 0 0 0.0000)
+		)
+		(property "Sheetname" "clock-generation"
+			(at 78.74 46.2784 0)
+			(effects
+				(font
+					(size 1.27 1.27)
+				)
+				(justify left bottom)
+			)
+		)
+		(property "Sheetfile" "clock-generation.kicad_sch"
+			(at 78.74 71.7046 0)
+			(effects
+				(font
+					(size 1.27 1.27)
+				)
+				(justify left top)
+			)
+		)
+		(instances
+			(project "dante-audio-board"
+				(path "/df100556-b288-4cb1-b69f-c0734132cb90"
+					(page "3")
+				)
+			)
+		)
+	)
+	(sheet_instances
+		(path "/"
+			(page "1")
+		)
+	)
 )

Commit message: wip
Other:
- added sheet audio-codec (audio-codec.kicad_sch)
- added sheet audio-connectors (audio-connectors.kicad_sch)
Changed lines of the file:
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@@
+		)
+	)
+	(sheet
+		(at 228.6 48.26)
+		(size 13.97 67.31)
+		(fields_autoplaced yes)
+		(stroke
+			(width 0.1524)
+			(type solid)
+		)
+		(fill
+			(color 0 0 0 0.0000)
+		)
+		(property "Sheetname" "audio-connectors"
+			(at 228.6 47.5484 0)
+			(effects
+				(font
+					(size 1.27 1.27)
+				)
+				(justify left bottom)
+			)
+		)
+		(property "Sheetfile" "audio-connectors.kicad_sch"
+			(at 228.6 116.1546 0)
+			(effects
+				(font
+					(size 1.27 1.27)
+				)
+				(justify left top)
+			)
+		)
+		(instances
+			(project "dante-audio-board"
+				(path "/df100556-b288-4cb1-b69f-c0734132cb90"
+					(page "5")
+				)
+			)
+		)
+	)
+	(sheet
+		(at 144.78 48.26)
+		(size 49.53 68.58)
+		(fields_autoplaced yes)
+		(stroke
+			(width 0.1524)
+			(type solid)
+		)
+		(fill
+			(color 0 0 0 0.0000)
+		)
+		(property "Sheetname" "audio-codec"
+			(at 144.78 47.5484 0)
+			(effects
+				(font
+					(size 1.27 1.27)
+				)
+				(justify left bottom)
+			)
+		)
+		(property "Sheetfile" "audio-codec.kicad_sch"
+			(at 144.78 117.4246 0)
+			(effects
+				(font
+					(size 1.27 1.27)
+				)
+				(justify left top)
+			)
+		)
+		(instances
+			(project "dante-audio-board"
+				(path "/df100556-b288-4cb1-b69f-c0734132cb90"
+					(page "4")
+				)
+			)
 		)
 	)

Commit message: wip
Other:
- sheet clock-generation ports: added COUNTER_FB, OSC_LRCLK, OSC_MCLK, OSC_SCLK, SCL, SDA; removed none
Changed lines of the file:
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@@
 	(generator "eeschema")
 	(generator_version "8.0")
-	(paper "A4")
+	(paper "USLetter")
 	(sheet
 		(at 46.99 46.99)
@@
 			)
 		)
+		(pin "SDA" bidirectional
+			(at 78.74 54.61 180)
+			(effects
+				(font
+					(size 1.27 1.27)
+				)
+				(justify left)
+			)
+		)
+		(pin "SCL" bidirectional
+			(at 78.74 57.15 180)
+			(effects
+				(font
+					(size 1.27 1.27)
+				)
+				(justify left)
+			)
+		)
+		(pin "OSC_SCLK" output
+			(at 119.38 52.07 0)
+			(effects
+				(font
+					(size 1.27 1.27)
+				)
+				(justify right)
+			)
+		)
+		(pin "OSC_LRCLK" output
+			(at 119.38 54.61 0)
+			(effects
+				(font
+					(size 1.27 1.27)
+				)
+				(justify right)
+			)
+		)
+		(pin "OSC_MCLK" output
+			(at 119.38 57.15 0)
+			(effects
+				(font
+					(size 1.27 1.27)
+				)
+				(justify right)
+			)
+		)
+		(pin "COUNTER_FB" output
+			(at 119.38 59.69 0)
+			(effects
+				(font
+					(size 1.27 1.27)
+				)
+				(justify right)
+			)
+		)
