File: clock-generation.kicad_sch (KiCad schematic)
At the start: 28 parts, among them U1 Si5351B-B-GM, U2 TPS79301-EP, U3 DAC53002RTER, Y1 7M-27.000MEEQ-T

Commit message: add 1-wire eeprom and a bit more
Parts:
- added R14: 10R, Resistor_SMD:R_0402_1005Metric, symbol Device:R
Connections:
- net at R9.2: now also U1.9 (CLK2); no longer U1.12 (CLK1)
- net at R10.2: now also U1.19 (CLK4); no longer U1.9 (CLK2)
- new net: R14.2, U1.12 (CLK1)
- new net TS: R14.1
- no-connect marks 4 -> 3
Other:
- moved on the sheet: R10, R9
Changed lines of the file:
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@@
 	)
 	(junction
-		(at 227.33 97.79)
+		(at 227.33 102.87)
 		(diameter 0)
 		(color 0 0 0 0)
@@
 	)
 	(junction
+		(at 227.33 97.79)
+		(diameter 0)
+		(color 0 0 0 0)
+	)
+	(junction
 		(at 139.7 95.25)
 		(diameter 0)
@@
 	)
 	(junction
-		(at 227.33 102.87)
+		(at 227.33 113.03)
 		(diameter 0)
 		(color 0 0 0 0)
@@
 	)
 	(no_connect
-		(at 212.09 113.03)
+		(at 212.09 118.11)
 	)
 	(no_connect
@@
 		(at 212.09 128.27)
 	)
-	(no_connect
-		(at 212.09 118.11)
-	)
 	(wire
 		(pts
@@
 	(wire
 		(pts
-			(xy 226.06 97.79) (xy 227.33 97.79)
+			(xy 226.06 102.87) (xy 227.33 102.87)
 		)
 		(stroke
@@
 	(wire
 		(pts
-			(xy 212.09 107.95) (xy 218.44 107.95)
-		)
-		(stroke
-			(width 0)
-			(type default)
-		)
-	)
-	(wire
-		(pts
 			(xy 115.57 128.27) (xy 121.92 128.27)
 		)
@@
 	(wire
 		(pts
+			(xy 212.09 97.79) (xy 218.44 97.79)
+		)
+		(stroke
+			(width 0)
+			(type default)
+		)
+	)
+	(wire
+		(pts
 			(xy 109.22 64.77) (xy 109.22 67.31)
 		)
@@
 	(wire
 		(pts
+			(xy 227.33 96.52) (xy 227.33 97.79)
+		)
+		(stroke
+			(width 0)
+			(type default)
+		)
+	)
+	(wire
+		(pts
 			(xy 77.47 97.79) (xy 77.47 100.33)
 		)
@@
 	(wire
 		(pts
+			(xy 212.09 107.95) (xy 218.44 107.95)
+		)
+		(stroke
+			(width 0)
+			(type default)
+		)
+	)
+	(wire
+		(pts
 			(xy 55.88 132.08) (xy 58.42 132.08)
 		)
@@
 	(wire
 		(pts
-			(xy 226.06 102.87) (xy 227.33 102.87)
+			(xy 226.06 113.03) (xy 227.33 113.03)
 		)
 		(stroke
@@
 	(wire
 		(pts
-			(xy 227.33 101.6) (xy 227.33 102.87)
+			(xy 227.33 111.76) (xy 227.33 113.03)
 		)
 		(stroke
@@
 	(wire
 		(pts
-			(xy 227.33 102.87) (xy 234.95 102.87)
+			(xy 227.33 113.03) (xy 234.95 113.03)
+		)
+		(stroke
+			(width 0)
+			(type default)
+		)
+	)
+	(wire
+		(pts
+			(xy 226.06 97.79) (xy 227.33 97.79)
 		)
 		(stroke
@@
 	(wire
 		(pts
-			(xy 212.09 97.79) (xy 218.44 97.79)
+			(xy 57.15 115.57) (xy 60.96 115.57)
 		)
 		(stroke
@@
 	(wire
 		(pts
-			(xy 57.15 115.57) (xy 60.96 115.57)
+			(xy 58.42 55.88) (xy 55.88 55.88)
 		)
 		(stroke
@@
 	(wire
 		(pts
-			(xy 58.42 55.88) (xy 55.88 55.88)
+			(xy 58.42 143.51) (xy 58.42 146.05)
 		)
 		(stroke
@@
 	(wire
 		(pts
-			(xy 58.42 143.51) (xy 58.42 146.05)
+			(xy 137.16 128.27) (xy 137.16 130.81)
 		)
 		(stroke
@@
 	(wire
 		(pts
-			(xy 137.16 128.27) (xy 137.16 130.81)
+			(xy 80.01 66.04) (xy 80.01 68.58)
 		)
 		(stroke
@@
 	(wire
 		(pts
-			(xy 80.01 66.04) (xy 80.01 68.58)
+			(xy 212.09 102.87) (xy 218.44 102.87)
 		)
 		(stroke
@@
 	(wire
 		(pts
-			(xy 227.33 96.52) (xy 227.33 97.79)
+			(xy 227.33 101.6) (xy 227.33 102.87)
 		)
 		(stroke
@@
 	(wire
 		(pts
+			(xy 212.09 113.03) (xy 218.44 113.03)
+		)
+		(stroke
+			(width 0)
+			(type default)
+		)
+	)
+	(wire
+		(pts
 			(xy 247.65 80.01) (xy 247.65 78.74)
 		)
@@
 	(wire
 		(pts
-			(xy 212.09 102.87) (xy 218.44 102.87)
+			(xy 227.33 102.87) (xy 234.95 102.87)
 		)
 		(stroke
@@
 	(wire
 		(pts
-			(xy 227.33 97.79) (xy 234.95 97.79)
+			(xy 168.91 118.11) (xy 181.61 118.11)
 		)
 		(stroke
@@
 	(wire
 		(pts
-			(xy 168.91 118.11) (xy 181.61 118.11)
+			(xy 92.71 69.85) (xy 92.71 72.39)
 		)
 		(stroke
@@
 	(wire
 		(pts
-			(xy 92.71 69.85) (xy 92.71 72.39)
+			(xy 55.88 55.88) (xy 55.88 52.07)
 		)
 		(stroke
@@
 	(wire
 		(pts
-			(xy 55.88 55.88) (xy 55.88 52.07)
+			(xy 177.8 128.27) (xy 177.8 130.81)
 		)
 		(stroke
@@
 	(wire
 		(pts
-			(xy 177.8 128.27) (xy 177.8 130.81)
+			(xy 139.7 100.33) (xy 139.7 95.25)
 		)
 		(stroke
@@
 	(wire
 		(pts
-			(xy 139.7 100.33) (xy 139.7 95.25)
+			(xy 227.33 97.79) (xy 234.95 97.79)
 		)
 		(stroke
@@
 	(hierarchical_label "OSC_LRCLK"
 		(shape output)
-		(at 234.95 97.79 0)
+		(at 234.95 102.87 0)
 		(fields_autoplaced yes)
 		(effects
@@
 	(hierarchical_label "OSC_MCLK"
 		(shape output)
-		(at 234.95 102.87 0)
+		(at 234.95 113.03 0)
 		(fields_autoplaced yes)
 		(effects
@@
 		)
 	)
+	(hierarchical_label "TS"
+		(shape output)
+		(at 234.95 97.79 0)
+		(fields_autoplaced yes)
+		(effects
+			(font
+				(size 1.27 1.27)
+			)
+			(justify left)
+		)
+	)
 	(hierarchical_label "SDA"
 		(shape bidirectional)
@@
 		(length 2.54)
 		(shape round)
-		(at 227.33 101.6 0)
+		(at 227.33 111.76 0)
 		(effects
 			(font
@@
 		)
 		(property "Netclass" "50ohm"
-			(at 227.838 100.838 0)
+			(at 227.838 110.998 0)
 			(effects
 				(font
@@
 		(length 2.54)
 		(shape round)
-		(at 227.33 96.52 0)
+		(at 227.33 101.6 0)
 		(effects
 			(font
@@
 		)
 		(property "Netclass" "50ohm"
-			(at 228.092 95.758 0)
+			(at 228.092 100.838 0)
 			(effects
 				(font
@@
 		(length 2.54)
 		(shape round)
+		(at 227.33 96.52 0)
+		(effects
+			(font
+				(size 1.27 1.27)
+			)
+			(justify left bottom)
+		)
+		(property "Netclass" "50ohm"
+			(at 228.092 95.758 0)
+			(effects
+				(font
+					(size 1.27 1.27)
+					(italic yes)
+				)
+				(justify left)
+			)
+		)
+	)
+	(netclass_flag ""
+		(length 2.54)
+		(shape round)
 		(at 227.33 91.44 0)
 		(effects
@@
 	(symbol
 		(lib_id "Device:R")
-		(at 222.25 97.79 270)
+		(at 222.25 102.87 270)
 		(unit 1)
 		(exclude_from_sim no)
@@
 		(dnp no)
 		(property "Reference" "R9"
-			(at 221.488 95.758 90)
+			(at 221.488 100.838 90)
 			(effects
 				(font
@@
 		)
 		(property "Value" "10R"
-			(at 221.996 97.79 90)
+			(at 221.996 102.87 90)
 			(effects
 				(font
@@
 		)
 		(property "Footprint" "Resistor_SMD:R_0402_1005Metric"
-			(at 222.25 96.012 90)
+			(at 222.25 101.092 90)
 			(effects
 				(font
@@
 		)
 		(property "Datasheet" "~"
-			(at 222.25 97.79 0)
+			(at 222.25 102.87 0)
 			(effects
 				(font
@@
 		)
 		(property "Description" "Resistor"
-			(at 222.25 97.79 0)
+			(at 222.25 102.87 0)
 			(effects
 				(font
@@
 	(symbol
 		(lib_id "Device:R")
-		(at 222.25 102.87 270)
+		(at 222.25 113.03 270)
 		(unit 1)
 		(exclude_from_sim no)
@@
 		(dnp no)
 		(property "Reference" "R10"
-			(at 221.742 100.584 90)
+			(at 221.742 110.744 90)
 			(effects
 				(font
@@
 		)
 		(property "Value" "10R"
-			(at 221.996 102.87 90)
+			(at 221.996 113.03 90)
 			(effects
 				(font
@@
 		)
 		(property "Footprint" "Resistor_SMD:R_0402_1005Metric"
-			(at 222.25 101.092 90)
+			(at 222.25 111.252 90)
 			(effects
 				(font
@@
 		)
 		(property "Datasheet" "~"
-			(at 222.25 102.87 0)
+			(at 222.25 113.03 0)
 			(effects
 				(font
@@
 		)
 		(property "Description" "Resistor"
-			(at 222.25 102.87 0)
+			(at 222.25 113.03 0)
 			(effects
 				(font
@@
 					(unit 1)
 				)
+			)
+		)
+	)
+	(symbol
+		(lib_id "Device:R")
+		(at 222.25 97.79 270)
+		(unit 1)
+		(exclude_from_sim no)
+		(in_bom yes)
+		(on_board yes)
+		(dnp no)
+		(property "Reference" "R14"
+			(at 221.488 95.758 90)
+			(effects
+				(font
+					(size 1.27 1.27)
+				)
+			)
+		)
+		(property "Value" "10R"
+			(at 221.996 97.79 90)
+			(effects
+				(font
+					(size 1.27 1.27)
+				)
+			)
+		)
+		(property "Footprint" "Resistor_SMD:R_0402_1005Metric"
+			(at 222.25 96.012 90)
+			(effects
+				(font
+					(size 1.27 1.27)
+				)
+				(hide yes)
+			)
+		)
+		(property "Datasheet" "~"
+			(at 222.25 97.79 0)
+			(effects
+				(font
+					(size 1.27 1.27)
+				)
+				(hide yes)
+			)
+		)
+		(property "Description" "Resistor"
+			(at 222.25 97.79 0)
+			(effects
+				(font
+					(size 1.27 1.27)
+				)
+				(hide yes)
+			)
+		)
+		(pin "2"
+		)
+		(pin "1"
+		)
+		(instances
+			(project "jkembedded-audio-board"
+				(path "/df100556-b288-4cb1-b69f-c0734132cb90/be7c4f40-c0c2-47f2-9c0c-8904af6555df"
+					(reference "R14")
+					(unit 1)
+				)

Commit message: add MSPM0
Parts:
- C9: footprint Capacitor_Tantalum_SMD:CP_EIA-6032-15_Kemet-U -> Capacitor_Tantalum_SMD:CP_EIA-3216-18_Kemet-A
Changed lines of the file:
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@@
 			)
 		)
-		(property "Footprint" "Capacitor_Tantalum_SMD:CP_EIA-6032-15_Kemet-U"
+		(property "Footprint" "Capacitor_Tantalum_SMD:CP_EIA-3216-18_Kemet-A"
 			(at 199.0852 77.47 0)
 			(effects

Commit message: add clickid
Parts:
- TP1: now not fitted; now left out of the parts list
Changed lines of the file:
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@@
 		(unit 1)
 		(exclude_from_sim no)
-		(in_bom yes)
+		(in_bom no)
 		(on_board yes)
-		(dnp no)
+		(dnp yes)
 		(fields_autoplaced yes)
 		(property "Reference" "TP1"

Commit message: add extra labels to MB and title. specify project in CI file and update to Kicad 8.0.8
Other:
- company: (none) -> JKEmbedded, LLC
- title: (none) -> JKEmbedded Audio Board
Changed lines of the file:
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@@
 	(generator_version "8.0")
 	(paper "USLetter")
+	(title_block
+		(title "JKEmbedded Audio Board")
+		(company "JKEmbedded, LLC")
+	)
 	(junction
 		(at 229.87 78.74)

Commit message: Resolved #2: Matched 4 clock outputs to expected by DEP
Parts:
- removed R14: 10R, Resistor_SMD:R_0402_1005Metric, symbol Device:R
Connections:
- net at R9.2: now also U1.12 (CLK1); no longer U1.9 (CLK2)
- net at R10.2: now also U1.9 (CLK2); no longer U1.19 (CLK4)
- no-connect marks 3 -> 4
Other:
- moved on the sheet: R10, R9
Changed lines of the file:
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@@
 	)
 	(junction
-		(at 227.33 102.87)
+		(at 227.33 97.79)
 		(diameter 0)
 		(color 0 0 0 0)
@@
 	)
 	(junction
-		(at 227.33 97.79)
-		(diameter 0)
-		(color 0 0 0 0)
-	)
-	(junction
 		(at 139.7 95.25)
 		(diameter 0)
@@
 	)
 	(junction
-		(at 227.33 113.03)
+		(at 227.33 102.87)
 		(diameter 0)
 		(color 0 0 0 0)
@@
 	)
 	(no_connect
+		(at 212.09 113.03)
+	)
+	(no_connect
 		(at 212.09 128.27)
 	)
@@
 	(wire
 		(pts
-			(xy 226.06 102.87) (xy 227.33 102.87)
+			(xy 226.06 97.79) (xy 227.33 97.79)
 		)
 		(stroke
@@
 	(wire
 		(pts
-			(xy 212.09 97.79) (xy 218.44 97.79)
-		)
-		(stroke
-			(width 0)
-			(type default)
-		)
-	)
-	(wire
-		(pts
 			(xy 109.22 64.77) (xy 109.22 67.31)
 		)
@@
 	(wire
 		(pts
-			(xy 227.33 96.52) (xy 227.33 97.79)
-		)
-		(stroke
-			(width 0)
-			(type default)
-		)
-	)
-	(wire
-		(pts
 			(xy 77.47 97.79) (xy 77.47 100.33)
 		)
@@
 	(wire
 		(pts
-			(xy 226.06 113.03) (xy 227.33 113.03)
+			(xy 226.06 102.87) (xy 227.33 102.87)
 		)
 		(stroke
@@
 	(wire
 		(pts
-			(xy 227.33 111.76) (xy 227.33 113.03)
+			(xy 227.33 101.6) (xy 227.33 102.87)
 		)
 		(stroke
@@
 	(wire
 		(pts
-			(xy 227.33 113.03) (xy 234.95 113.03)
-		)
-		(stroke
-			(width 0)
-			(type default)
-		)
-	)
-	(wire
-		(pts
-			(xy 226.06 97.79) (xy 227.33 97.79)
+			(xy 227.33 102.87) (xy 234.95 102.87)
 		)
 		(stroke
@@
 	(wire
 		(pts
-			(xy 212.09 102.87) (xy 218.44 102.87)
+			(xy 212.09 97.79) (xy 218.44 97.79)
 		)
 		(stroke
@@
 	(wire
 		(pts
-			(xy 227.33 101.6) (xy 227.33 102.87)
+			(xy 227.33 96.52) (xy 227.33 97.79)
 		)
 		(stroke
@@
 	(wire
 		(pts
-			(xy 212.09 113.03) (xy 218.44 113.03)
+			(xy 212.09 102.87) (xy 218.44 102.87)
 		)
 		(stroke
@@
 	(wire
 		(pts
-			(xy 227.33 102.87) (xy 234.95 102.87)
+			(xy 227.33 97.79) (xy 234.95 97.79)
 		)
 		(stroke
@@
 	(wire
 		(pts
-			(xy 227.33 97.79) (xy 234.95 97.79)
-		)
-		(stroke
-			(width 0)
-			(type default)
-		)
-	)
-	(wire
-		(pts
 			(xy 143.51 128.27) (xy 137.16 128.27)
 		)
@@
 	(hierarchical_label "OSC_LRCLK"
 		(shape output)
-		(at 234.95 102.87 0)
+		(at 234.95 97.79 0)
 		(effects
 			(font
@@
 	(hierarchical_label "OSC_MCLK"
 		(shape output)
-		(at 234.95 113.03 0)
+		(at 234.95 102.87 0)
 		(effects
 			(font
@@
 		)
 	)
-	(hierarchical_label "TS"
-		(shape output)
-		(at 234.95 97.79 0)
-		(effects
-			(font
-				(size 1.27 1.27)
-			)
-			(justify left)
-		)
-	)
 	(hierarchical_label "SDA"
 		(shape bidirectional)
@@
 		(length 2.54)
 		(shape round)
-		(at 227.33 111.76 0)
+		(at 227.33 101.6 0)
 		(effects
 			(font
@@
 		)
 		(property "Netclass" "50ohm"
-			(at 227.838 110.998 0)
+			(at 227.838 100.838 0)
 			(effects
 				(font
@@
 		(length 2.54)
 		(shape round)
-		(at 227.33 101.6 0)
+		(at 227.33 96.52 0)
 		(effects
 			(font
@@
 		)
 		(property "Netclass" "50ohm"
-			(at 228.092 100.838 0)
+			(at 228.092 95.758 0)
 			(effects
 				(font
@@
 		(length 2.54)
 		(shape round)
-		(at 227.33 96.52 0)
-		(effects
-			(font
-				(size 1.27 1.27)
-			)
-			(justify left bottom)
-		)
-		(property "Netclass" "50ohm"
-			(at 228.092 95.758 0)
-			(effects
-				(font
-					(size 1.27 1.27)
-					(italic yes)
-				)
-				(justify left)
-			)
-		)
-	)
-	(netclass_flag ""
-		(length 2.54)
-		(shape round)
 		(at 227.33 91.44 0)
 		(effects
@@
 	(symbol
 		(lib_id "Device:R")
-		(at 222.25 102.87 270)
+		(at 222.25 97.79 270)
 		(unit 1)
 		(exclude_from_sim no)
@@
 		(dnp no)
 		(property "Reference" "R9"
-			(at 221.488 100.838 90)
+			(at 221.488 95.758 90)
 			(effects
 				(font
@@
 		)
 		(property "Value" "10R"
-			(at 221.996 102.87 90)
+			(at 221.996 97.79 90)
 			(effects
 				(font
@@
 		)
 		(property "Footprint" "Resistor_SMD:R_0402_1005Metric"
-			(at 222.25 101.092 90)
+			(at 222.25 96.012 90)
 			(effects
 				(font
@@
 		)
 		(property "Datasheet" "~"
-			(at 222.25 102.87 0)
+			(at 222.25 97.79 0)
 			(effects
 				(font
@@
 		)
 		(property "Description" "Resistor"
-			(at 222.25 102.87 0)
+			(at 222.25 97.79 0)
 			(effects
 				(font
@@
 	(symbol
 		(lib_id "Device:R")
-		(at 222.25 113.03 270)
+		(at 222.25 102.87 270)
 		(unit 1)
 		(exclude_from_sim no)
@@
 		(dnp no)
 		(property "Reference" "R10"
-			(at 221.742 110.744 90)
+			(at 221.742 100.584 90)
 			(effects
 				(font
@@
 		)
 		(property "Value" "10R"
-			(at 221.996 113.03 90)
+			(at 221.996 102.87 90)
 			(effects
 				(font
@@
 		)
 		(property "Footprint" "Resistor_SMD:R_0402_1005Metric"
-			(at 222.25 111.252 90)
+			(at 222.25 101.092 90)
 			(effects
 				(font
@@
 		)
 		(property "Datasheet" "~"
-			(at 222.25 113.03 0)
+			(at 222.25 102.87 0)
 			(effects
 				(font
@@
 		)
 		(property "Description" "Resistor"
-			(at 222.25 113.03 0)
+			(at 222.25 102.87 0)
 			(effects
 				(font
@@
 					(unit 1)
 				)
-			)
-		)
-	)
-	(symbol
-		(lib_id "Device:R")
-		(at 222.25 97.79 270)
-		(unit 1)
-		(exclude_from_sim no)
-		(in_bom yes)
-		(on_board yes)
-		(dnp no)
-		(property "Reference" "R14"
-			(at 221.488 95.758 90)
-			(effects
-				(font
-					(size 1.27 1.27)
-				)
-			)
-		)
-		(property "Value" "10R"
-			(at 221.996 97.79 90)
-			(effects
-				(font
-					(size 1.27 1.27)
-				)
-			)
-		)
-		(property "Footprint" "Resistor_SMD:R_0402_1005Metric"
-			(at 222.25 96.012 90)
-			(effects
-				(font
-					(size 1.27 1.27)
-				)
-				(hide yes)
-			)
-		)
-		(property "Datasheet" "~"
-			(at 222.25 97.79 0)
-			(effects
-				(font
-					(size 1.27 1.27)
-				)
-				(hide yes)
-			)
-		)
-		(property "Description" "Resistor"
-			(at 222.25 97.79 0)
-			(effects
-				(font
-					(size 1.27 1.27)
-				)
-				(hide yes)
-			)
-		)
-		(pin "2"
-		)
-		(pin "1"
-		)
-		(instances
-			(project "jkembedded-audio-board"
-				(path "/df100556-b288-4cb1-b69f-c0734132cb90/be7c4f40-c0c2-47f2-9c0c-8904af6555df"
-					(reference "R14")
-					(unit 1)
-				)
